File: hardware/power.kicad_sch (KiCad schematic)
At the start: 33 parts, among them U1 RY1303, U2 AP2112K-1.8, U3 AP2112K-1.8, U4 APX803-29SAG-7, U5 TPS2051BDBVR

Commit message: 原理圖十一頁全部寫進專案,ERC 歸零
關掉 KiCad 之後執行 run_all.py --apply,23 步全過。

關閉前先確認過未存檔的修改是什麼:
  KiCad 標題有 * 標記,但比對 .history(KiCad 自己的 autosave repo)
  與 HEAD 的差異只有 10 行,而且全是視覺層面 ——
  一條裝飾用分隔線的端點差 0.76mm、一顆 GND 符號的文字標籤位置。
  沒有任何元件、接線、net 名稱、腳位的改變。
  而且 .history 那份(15:50 autosave)比 HEAD(15:51 commit)還舊,
  磁碟上的就是最新版。沒有東西遺失。

寫進專案的內容
  新增 8 張子頁:display / hdmi / mipi / net / usb / storage / header / audio
  mcu 頁補 unit 6/7 接線、兩顆晶振、23 顆逐腳去耦
  power 頁補 4 個 PWR_FLAG
  修掉手畫頁殘留:兩段 1.27mm 殘線、AGND 線尾沒放接地符號、
  排針串接電阻與兩顆 IC 的 footprint
  PG12/PG14/PG4 改名為 HDMI_INT_N / HDMI_PD / PANEL_RESET_N
  產生 T113-S3 的 eLQFP128 footprint(內建件 + EPAD + thermal via)

驗證(真實專案,非副本)
  ERC                0 errors · 0 warnings
  check_schematic    0 errors · 0 warnings
  check_power_rails  全部通過
  209 顆元件 · 253 條 net · 11 頁 · 缺 footprint 0

接下來是 PCB layout,那是使用者的部分。

Co-Authored-By: Claude Opus 5 <noreply@anthropic.com>
Claude-Session: https://claude.ai/code/session_01HtGUWSQFey6W2g2grqgTMR
Parts:
- U1: footprint (none) -> Package_DFN_QFN:UQFN-20-1EP_3x3mm_P0.4mm_EP1.7x1.7mm_ThermalVias
Other:
- note added: "PWR_FLAG —— 給 ERC 看的，不是真元件"
- note added: "⚠ 只能用在確實有電的地方 —— 拿它蓋掉真的沒接的軌等於把安全網剪掉。"
- note added: "所以 ERC 在輸出節點上找不到任何 power_out 腳，判定「沒人驅動」。"
- note added: "降壓器的輸出走 SW 腳 ->[電感]-> 輸出節點，電感是被動件，"
