File: hardware/power.kicad_sch (KiCad schematic)
At the start: 33 parts, among them U1 RY1303, U2 AP2112K-1.8, U3 AP2112K-1.8, U4 APX803-29SAG-7, U5 TPS2051BDBVR

Commit message: 還原圖紙到生成前,準備用修好的腳本重跑
Parts:
- U1: footprint Package_DFN_QFN:UQFN-20-1EP_3x3mm_P0.4mm_EP1.7x1.7mm_ThermalVias -> (none)
Other:
- note removed: "PWR_FLAG —— 給 ERC 看的，不是真元件"
- note removed: "⚠ 只能用在確實有電的地方 —— 拿它蓋掉真的沒接的軌等於把安全網剪掉。"
- note removed: "所以 ERC 在輸出節點上找不到任何 power_out 腳，判定「沒人驅動」。"
- note removed: "降壓器的輸出走 SW 腳 ->[電感]-> 輸出節點，電感是被動件，"

Commit message: wip
Parts:
- U1: footprint (none) -> Package_DFN_QFN:UQFN-20-1EP_3x3mm_P0.4mm_EP1.7x1.7mm_ThermalVias
Other:
- note added: "PWR_FLAG —— 給 ERC 看的，不是真元件"
- note added: "⚠ 只能用在確實有電的地方 —— 拿它蓋掉真的沒接的軌等於把安全網剪掉。"
- note added: "所以 ERC 在輸出節點上找不到任何 power_out 腳，判定「沒人驅動」。"
- note added: "降壓器的輸出走 SW 腳 ->[電感]-> 輸出節點，電感是被動件，"

Commit message: 還原,最終完整重跑
Parts:
- U1: footprint Package_DFN_QFN:UQFN-20-1EP_3x3mm_P0.4mm_EP1.7x1.7mm_ThermalVias -> (none)
Other:
- note removed: "PWR_FLAG —— 給 ERC 看的，不是真元件"
- note removed: "⚠ 只能用在確實有電的地方 —— 拿它蓋掉真的沒接的軌等於把安全網剪掉。"
- note removed: "所以 ERC 在輸出節點上找不到任何 power_out 腳，判定「沒人驅動」。"
- note removed: "降壓器的輸出走 SW 腳 ->[電感]-> 輸出節點，電感是被動件，"

Commit message: wip
Parts:
- U1: footprint (none) -> Package_DFN_QFN:UQFN-20-1EP_3x3mm_P0.4mm_EP1.7x1.7mm_ThermalVias
Other:
- note added: "PWR_FLAG —— 給 ERC 看的，不是真元件"
- note added: "⚠ 只能用在確實有電的地方 —— 拿它蓋掉真的沒接的軌等於把安全網剪掉。"
- note added: "所以 ERC 在輸出節點上找不到任何 power_out 腳，判定「沒人驅動」。"
- note added: "降壓器的輸出走 SW 腳 ->[電感]-> 輸出節點，電感是被動件，"

Commit message: 還原,準備最終完整重跑
Parts:
- U1: footprint Package_DFN_QFN:UQFN-20-1EP_3x3mm_P0.4mm_EP1.7x1.7mm_ThermalVias -> (none)
Other:
- note removed: "PWR_FLAG —— 給 ERC 看的，不是真元件"
- note removed: "⚠ 只能用在確實有電的地方 —— 拿它蓋掉真的沒接的軌等於把安全網剪掉。"
- note removed: "所以 ERC 在輸出節點上找不到任何 power_out 腳，判定「沒人驅動」。"
- note removed: "降壓器的輸出走 SW 腳 ->[電感]-> 輸出節點，電感是被動件，"
