File: hardware/power.kicad_sch (KiCad schematic)
At the start: 33 parts, among them U1 RY1303, U2 AP2112K-1.8, U3 AP2112K-1.8, U4 APX803-29SAG-7, U5 TPS2051BDBVR

Commit message: 佈線前置檢查:修掉三件會擋住或拖累佈線的事
ERC 歸零不等於能開始佈線。再問一次「丟進 PCB 編輯器,佈線工具真的能用嗎」,
答案是當時還不能。

★ ① ERC 完全不看「原理圖 ↔ footprint」的對應
   TP9/TP10/TP11 的 footprint 被設成繼電器(手畫時選錯)
     測試點只有 pad 1,繼電器的焊盤編號是 11/12/14/21/22/24/A1/A2
   Y3 用 4 腳的 Crystal_GND24 符號配 2 腳的 3215 封裝
   兩個都通過 ERC、也通過「有沒有填 footprint」「檔案在不在」的檢查 ——
   原理圖上完全正常,只有把兩邊擺在一起比才看得出來。Update PCB 會直接卡住。
   新增 check_footprints.py 並列入 run_all。

★ ② 差分對命名不符合 KiCad 的識別規則
   KiCad 用 net 名稱字尾 _P/_N(或 +/-)判斷「這兩條是一對」。
     ✓ TMDS_D0_P / MDI0_P      認得
     ✗ DSI_D0P                 字尾是 0P
     ✗ USB0_DP                 字尾是 DP
   後果:差分對佈線工具與對內等長調整,對 MIPI 與 USB 全部不能用 ——
   而 MIPI 差分佈線正是這塊板最主要的練習目標。
   全部改名,現在 17 組差分對(MIPI 5 · TMDS 4 · USB 6 · ETH 2)全部合規。
   mcu 頁的 DSI 標籤是手畫的,走 rename_nets.py 的三道保險。

③ netclass 建好六類分組,線寬刻意留空
   MIPI_DSI 10 · TMDS 8 · USB_HS 12 · ETH_MDI 4 · RGB_LCD 22 · POWER 15
   不填線寬是因為 005 §2:必須用 JLCPCB 的阻抗計算器回算,不能自行假設。
   先分類的好處是回算後在一個地方改數字,全部走線跟著改。

最終驗證(真實專案,從乾淨狀態完整重跑 27 步)
  ERC                0 errors · 0 warnings
  check_schematic    0 errors · 0 warnings
  check_power_rails  全部通過
  check_footprints   209 顆元件腳號全部對得上焊盤
  11 頁 · 253 條 net

Co-Authored-By: Claude Opus 5 <noreply@anthropic.com>
Claude-Session: https://claude.ai/code/session_01HtGUWSQFey6W2g2grqgTMR
Parts:
- U1: footprint (none) -> Package_DFN_QFN:UQFN-20-1EP_3x3mm_P0.4mm_EP1.7x1.7mm_ThermalVias
Other:
- note added: "PWR_FLAG —— 給 ERC 看的，不是真元件"
- note added: "⚠ 只能用在確實有電的地方 —— 拿它蓋掉真的沒接的軌等於把安全網剪掉。"
- note added: "所以 ERC 在輸出節點上找不到任何 power_out 腳，判定「沒人驅動」。"
- note added: "降壓器的輸出走 SW 腳 ->[電感]-> 輸出節點，電感是被動件，"
