File: hardware/T113-DEV-V1.kicad_sch (KiCad schematic)
At the start: 0 parts

Commit message: 還原圖紙到生成前,準備用修好的腳本重跑
Other:
- removed sheet USB 與開機
- removed sheet 儲存
- removed sheet 排針
- removed sheet 網路
- removed sheet 音訊
- removed sheet 顯示 · ADV7511
- removed sheet 顯示 · HDMI 座
- removed sheet 顯示 · MIPI DSI
