File: hardware/T113-DEV-V1.kicad_sch (KiCad schematic)
At the start: 0 parts

Commit message: 還原,最終重跑
Other:
- removed sheet USB 與開機
- removed sheet 儲存
- removed sheet 排針
- removed sheet 網路
- removed sheet 音訊
- removed sheet 顯示 · ADV7511
- removed sheet 顯示 · HDMI 座
- removed sheet 顯示 · MIPI DSI

Commit message: wip
Other:
- added sheet USB 與開機 (usb.kicad_sch)
- added sheet 儲存 (storage.kicad_sch)
- added sheet 排針 (header.kicad_sch)
- added sheet 網路 (net.kicad_sch)
- added sheet 音訊 (audio.kicad_sch)
- added sheet 顯示 · ADV7511 (display.kicad_sch)
- added sheet 顯示 · HDMI 座 (hdmi.kicad_sch)
- added sheet 顯示 · MIPI DSI (mipi.kicad_sch)

Commit message: 還原,最終完整重跑
Other:
- removed sheet USB 與開機
- removed sheet 儲存
- removed sheet 排針
- removed sheet 網路
- removed sheet 音訊
- removed sheet 顯示 · ADV7511
- removed sheet 顯示 · HDMI 座
- removed sheet 顯示 · MIPI DSI
