File: hardware/T113-DEV-V1.kicad_sch (KiCad schematic)
At the start: 0 parts

Commit message: 佈線前置總驗收通過;修掉根圖紙上四張子頁蓋住 Main Chip 的問題
這一輪做了四項之前沒驗過的檢查,抓到一個排版問題。

★ 根圖紙上「Main Chip」被四張新子頁蓋住
   new_sheet.py 原本用「第 n 張放第 n 格」算位置,但電源與 Main Chip
   是手動放的,位置不在格線上,而且 Main Chip 比標準格子大(100x71mm)。
   結果 MIPI/網路/排針/音訊四張疊在它上面 —— 電氣沒影響,
   但根圖紙上點不到被蓋住的方塊,很難用。
   改成:讀出既有所有方塊的矩形,逐一試候選位置,挑第一個不重疊的。
   順手修掉 SLOTS 自己的 bug(236.22+88.9 > 320.04,第二三格會互撞)。

其餘三項新檢查都過
   BOM 匯出 209 列,DNP 標記正確(R65/R68/R78 = strap 不焊的那三顆)
   跨頁 UUID 3830 個,重複 0
   page 編號無重複

佈線前置總驗收(真實專案,從乾淨狀態完整重跑 27 步)
   ① ERC                0 errors · 0 warnings
   ② check_schematic    0 errors · 0 warnings
   ③ check_power_rails  全部通過
   ④ check_footprints   209 顆元件腳號全部對得上焊盤
   ⑤ BOM 匯出           209 列
   ⑥ 根圖紙             10 張子頁,方塊重疊 0
   ⑦ 元素 UUID          3830 個,重複 0
   ⑧ netclass           六類分組就位(線寬待 JLCPCB 阻抗回算)

可以 Update PCB from Schematic 了。

Co-Authored-By: Claude Opus 5 <noreply@anthropic.com>
Claude-Session: https://claude.ai/code/session_01HtGUWSQFey6W2g2grqgTMR
Other:
- added sheet USB 與開機 (usb.kicad_sch)
- added sheet 儲存 (storage.kicad_sch)
- added sheet 排針 (header.kicad_sch)
- added sheet 網路 (net.kicad_sch)
- added sheet 音訊 (audio.kicad_sch)
- added sheet 顯示 · ADV7511 (display.kicad_sch)
- added sheet 顯示 · HDMI 座 (hdmi.kicad_sch)
- added sheet 顯示 · MIPI DSI (mipi.kicad_sch)
