File: hardware/mcu.kicad_sch (KiCad schematic)
At the start: 76 parts, among them U6 T113-S3, Y2 24MHz, Y3 32.768kHz

Commit message: 還原,準備最終完整重跑
Parts:
- removed C20, C21: 0.1uF, Capacitor_SMD:C_0603_1608Metric, symbol Device:C
- removed C43, C44, C45, C46: 22pF, Capacitor_SMD:C_0603_1608Metric, symbol Device:C
- removed C62, C63, C64, C65, C66, C68, C69, C72, C73, C74, C75, C76, C77, C78, C79, C80, C81, C82, C83, C84: 100nF, Capacitor_SMD:C_0603_1608Metric, symbol Device:C
- removed C67, C70: 10uF, Capacitor_SMD:C_0805_2012Metric, symbol Device:C
- removed C71: 2.2uF, Capacitor_SMD:C_0603_1608Metric, symbol Device:C
- removed R37, R38: 33R, Resistor_SMD:R_0603_1608Metric, symbol Device:R
- removed R39: 240R, Resistor_SMD:R_0603_1608Metric, symbol Device:R
- removed Y2: 24MHz, Crystal:Crystal_SMD_2520-4Pin_2.5x2.0mm, symbol Device:Crystal_GND24
- removed Y3: 32.768kHz, Crystal:Crystal_SMD_3215-2Pin_3.2x1.5mm, symbol Device:Crystal
- R20, R21, R22, R23, R24, R25, R26, R27, R28, R29, R30, R31, R32, R33, R34, R35, R36: footprint Resistor_SMD:R_0603_1608Metric -> (none)
- TP10, TP11, TP9: footprint TestPoint:TestPoint_Pad_D1.5mm -> Relay_THT:Relay_DPDT_Schrack-RT2-FormC_RM5mm
- U6: footprint T113-DEV-V1:eLQFP-128_14x14mm_P0.4mm_EP5.72x5.72mm_ThermalVias -> (none)
Connections:
- net GND: no longer C18.1, C19.1, R36.1, U6.91 (AGND)
- net DSI_CK_N renamed DSI_CKN
- net DSI_CK_P renamed DSI_CKP
- net DSI_D0_N renamed DSI_D0N
- net DSI_D0_P renamed DSI_D0P
- net DSI_D1_N renamed DSI_D1N
- net DSI_D1_P renamed DSI_D1P
- net DSI_D2_N renamed DSI_D2N
- net DSI_D2_P renamed DSI_D2P
- net DSI_D3_N renamed DSI_D3N
- net DSI_D3_P renamed DSI_D3P
- net DXIN: no longer names the net of U6.23 (DXIN)
- net DXOUT: no longer names the net of U6.22 (DXOUT)
- net HDMI_INT_N renamed HDR_GPIO8
- net HDMI_PD renamed HDR_GPIO9
- net HP_FB: no longer names the net of U6.100 (HPOUTFB)
- net PANEL_RESET_N renamed HDR_GPIO7
- net SYS_RESET_N: no longer names the net of U6.27 (RESET)
- net USB0_D_N: no longer names the net of U6.114 (USB0-DM)
- net USB0_D_P: no longer names the net of U6.115 (USB0-DP)
- net USB1_D_N: no longer names the net of U6.113 (USB1-DM)
- net USB1_D_P: no longer names the net of U6.112 (USB1-DP)
- net X32KIN: no longer names the net of U6.25 (X32KIN)
- net X32KOUT: no longer names the net of U6.24 (X32KOUT)
- new net: C18.1, C19.1, R36.1, U6.91 (AGND)
- no-connect marks 18 -> 0
Other:
- note removed: "T113-S3 的逐腳去耦（2026-10-10 補；mcu 頁手畫時漏了）"
- note removed: "★ 真正決定效果的是 layout：每一顆要貼著它負責的那支腳、via 直接下地平面。"
- note removed: "擺遠了就只是 BOM 上多幾顆料（概念 08）。"
- note removed: "每一條軌「幾支電源腳就幾顆 0.1uF」，核心與 DDR 另加 10uF 的本地 bulk。"
