File: hardware/mcu.kicad_sch (KiCad schematic)
At the start: 42 parts, among them U6 T113-S3

Commit message: 佈線前置檢查:修掉三件會擋住或拖累佈線的事
ERC 歸零不等於能開始佈線。再問一次「丟進 PCB 編輯器,佈線工具真的能用嗎」,
答案是當時還不能。

★ ① ERC 完全不看「原理圖 ↔ footprint」的對應
   TP9/TP10/TP11 的 footprint 被設成繼電器(手畫時選錯)
     測試點只有 pad 1,繼電器的焊盤編號是 11/12/14/21/22/24/A1/A2
   Y3 用 4 腳的 Crystal_GND24 符號配 2 腳的 3215 封裝
   兩個都通過 ERC、也通過「有沒有填 footprint」「檔案在不在」的檢查 ——
   原理圖上完全正常,只有把兩邊擺在一起比才看得出來。Update PCB 會直接卡住。
   新增 check_footprints.py 並列入 run_all。

★ ② 差分對命名不符合 KiCad 的識別規則
   KiCad 用 net 名稱字尾 _P/_N(或 +/-)判斷「這兩條是一對」。
     ✓ TMDS_D0_P / MDI0_P      認得
     ✗ DSI_D0P                 字尾是 0P
     ✗ USB0_DP                 字尾是 DP
   後果:差分對佈線工具與對內等長調整,對 MIPI 與 USB 全部不能用 ——
   而 MIPI 差分佈線正是這塊板最主要的練習目標。
   全部改名,現在 17 組差分對(MIPI 5 · TMDS 4 · USB 6 · ETH 2)全部合規。
   mcu 頁的 DSI 標籤是手畫的,走 rename_nets.py 的三道保險。

③ netclass 建好六類分組,線寬刻意留空
   MIPI_DSI 10 · TMDS 8 · USB_HS 12 · ETH_MDI 4 · RGB_LCD 22 · POWER 15
   不填線寬是因為 005 §2:必須用 JLCPCB 的阻抗計算器回算,不能自行假設。
   先分類的好處是回算後在一個地方改數字,全部走線跟著改。

最終驗證(真實專案,從乾淨狀態完整重跑 27 步)
  ERC                0 errors · 0 warnings
  check_schematic    0 errors · 0 warnings
  check_power_rails  全部通過
  check_footprints   209 顆元件腳號全部對得上焊盤
  11 頁 · 253 條 net

Co-Authored-By: Claude Opus 5 <noreply@anthropic.com>
Claude-Session: https://claude.ai/code/session_01HtGUWSQFey6W2g2grqgTMR
Parts:
- added C20, C21: 0.1uF, Capacitor_SMD:C_0603_1608Metric, symbol Device:C
- added C43, C44, C45, C46: 22pF, Capacitor_SMD:C_0603_1608Metric, symbol Device:C
- added C62, C63, C64, C65, C66, C68, C69, C72, C73, C74, C75, C76, C77, C78, C79, C80, C81, C82, C83, C84: 100nF, Capacitor_SMD:C_0603_1608Metric, symbol Device:C
- added C67, C70: 10uF, Capacitor_SMD:C_0805_2012Metric, symbol Device:C
- added C71: 2.2uF, Capacitor_SMD:C_0603_1608Metric, symbol Device:C
- added R37, R38: 33R, Resistor_SMD:R_0603_1608Metric, symbol Device:R
- added R39: 240R, Resistor_SMD:R_0603_1608Metric, symbol Device:R
- added Y2: 24MHz, Crystal:Crystal_SMD_2520-4Pin_2.5x2.0mm, symbol Device:Crystal_GND24
- added Y3: 32.768kHz, Crystal:Crystal_SMD_3215-2Pin_3.2x1.5mm, symbol Device:Crystal
- R20, R21, R22, R23, R24, R25, R26, R27, R28, R29, R30, R31, R32, R33, R34, R35, R36: footprint (none) -> Resistor_SMD:R_0603_1608Metric
- TP10, TP11, TP9: footprint Relay_THT:Relay_DPDT_Schrack-RT2-FormC_RM5mm -> TestPoint:TestPoint_Pad_D1.5mm
- U6: footprint (none) -> T113-DEV-V1:eLQFP-128_14x14mm_P0.4mm_EP5.72x5.72mm_ThermalVias
Connections:
- net +0V9: now also C62.1, C63.1, C64.1, C65.1, C66.1, C67.1
- net +1V5: now also C68.1, C69.1, C70.1
- net +1V8_AUDIO: now also C71.1, C72.1, C73.1
- net +1V8_SOC: now also C74.1, C75.1, C76.1, C77.1, C78.1
- net +3V3: now also C79.1, C80.1, C81.1, C82.1, C83.1, C84.1
- net GND: now also C18.1, C19.1, R36.1, U6.91 (AGND), C43.2, C44.2, C45.2, C46.2, C62.2, C63.2, C64.2, C65.2, C66.2, C67.2, C68.2, C69.2, C70.2, C71.2, C72.2, C73.2, C74.2, C75.2, C76.2, C77.2, C78.2, C79.2, C80.2, C81.2, C82.2, C83.2, C84.2, R39.1, Y2.2 (G), Y2.4 (G)
- net HP_FB: now reaches U6.100 (HPOUTFB)
- net at U6.98 (HPOUTR): now also R38.1
- net at U6.99 (HPOUTL): now also R37.1
- net USB1_D_P: now reaches U6.112 (USB1-DP)
- net USB1_D_N: now reaches U6.113 (USB1-DM)
- net USB0_D_N: now reaches U6.114 (USB0-DM)
- net USB0_D_P: now reaches U6.115 (USB0-DP)
- net DXOUT: now reaches U6.22 (DXOUT)
- net DXOUT: now also C44.1, Y2.3
- net DXIN: now reaches U6.23 (DXIN)
- net DXIN: now also C43.1, Y2.1
- net X32KOUT: now reaches U6.24 (X32KOUT)
- net X32KOUT: now also C46.1, Y3.2
- net X32KIN: now reaches U6.25 (X32KIN)
- net X32KIN: now also C45.1, Y3.1
- net SYS_RESET_N: now reaches U6.27 (RESET)
- net at U6.47 (DZQ): now also R39.2
- net DSI_CKN renamed DSI_CK_N
- net DSI_CKP renamed DSI_CK_P
- net DSI_D0N renamed DSI_D0_N
- net DSI_D0P renamed DSI_D0_P
- net DSI_D1N renamed DSI_D1_N
- net DSI_D1P renamed DSI_D1_P
- net DSI_D2N renamed DSI_D2_N
- net DSI_D2P renamed DSI_D2_P
- net DSI_D3N renamed DSI_D3_N
- net DSI_D3P renamed DSI_D3_P
- net HDR_GPIO7 renamed PANEL_RESET_N
- net HDR_GPIO8 renamed HDMI_INT_N
- net HDR_GPIO9 renamed HDMI_PD
- new net: C20.1, R37.2
- new net: C21.1, R38.2
- new net HP_L: C20.2
- new net HP_R: C21.2
- no-connect marks 0 -> 18
Other:
- note added: "T113-S3 的逐腳去耦（2026-10-10 補；mcu 頁手畫時漏了）"
- note added: "★ 真正決定效果的是 layout：每一顆要貼著它負責的那支腳、via 直接下地平面。"
- note added: "擺遠了就只是 BOM 上多幾顆料（概念 08）。"
- note added: "每一條軌「幾支電源腳就幾顆 0.1uF」，核心與 DDR 另加 10uF 的本地 bulk。"
