File: hardware/mcu.kicad_sch (KiCad schematic)
At the start: 76 parts, among them U6 T113-S3, Y2 24MHz, Y3 32.768kHz

Commit message: 還原,最終重跑
Parts:
- removed C20, C21: 0.1uF, Capacitor_SMD:C_0603_1608Metric, symbol Device:C
- removed C43, C44, C45, C46: 22pF, Capacitor_SMD:C_0603_1608Metric, symbol Device:C
- removed C62, C63, C64, C65, C66, C68, C69, C72, C73, C74, C75, C76, C77, C78, C79, C80, C81, C82, C83, C84: 100nF, Capacitor_SMD:C_0603_1608Metric, symbol Device:C
- removed C67, C70: 10uF, Capacitor_SMD:C_0805_2012Metric, symbol Device:C
- removed C71: 2.2uF, Capacitor_SMD:C_0603_1608Metric, symbol Device:C
- removed R37, R38: 33R, Resistor_SMD:R_0603_1608Metric, symbol Device:R
- removed R39: 240R, Resistor_SMD:R_0603_1608Metric, symbol Device:R
- removed Y2: 24MHz, Crystal:Crystal_SMD_2520-4Pin_2.5x2.0mm, symbol Device:Crystal_GND24
- removed Y3: 32.768kHz, Crystal:Crystal_SMD_3215-2Pin_3.2x1.5mm, symbol Device:Crystal
- R20, R21, R22, R23, R24, R25, R26, R27, R28, R29, R30, R31, R32, R33, R34, R35, R36: footprint Resistor_SMD:R_0603_1608Metric -> (none)
- TP10, TP11, TP9: footprint TestPoint:TestPoint_Pad_D1.5mm -> Relay_THT:Relay_DPDT_Schrack-RT2-FormC_RM5mm
- U6: footprint T113-DEV-V1:eLQFP-128_14x14mm_P0.4mm_EP5.72x5.72mm_ThermalVias -> (none)
Connections:
- net GND: no longer C18.1, C19.1, R36.1, U6.91 (AGND)
- net DSI_CK_N renamed DSI_CKN
- net DSI_CK_P renamed DSI_CKP
- net DSI_D0_N renamed DSI_D0N
- net DSI_D0_P renamed DSI_D0P
- net DSI_D1_N renamed DSI_D1N
- net DSI_D1_P renamed DSI_D1P
- net DSI_D2_N renamed DSI_D2N
- net DSI_D2_P renamed DSI_D2P
- net DSI_D3_N renamed DSI_D3N
- net DSI_D3_P renamed DSI_D3P
- net DXIN: no longer names the net of U6.23 (DXIN)
- net DXOUT: no longer names the net of U6.22 (DXOUT)
- net HDMI_INT_N renamed HDR_GPIO8
- net HDMI_PD renamed HDR_GPIO9
- net HP_FB: no longer names the net of U6.100 (HPOUTFB)
- net PANEL_RESET_N renamed HDR_GPIO7
- net SYS_RESET_N: no longer names the net of U6.27 (RESET)
- net USB0_D_N: no longer names the net of U6.114 (USB0-DM)
- net USB0_D_P: no longer names the net of U6.115 (USB0-DP)
- net USB1_D_N: no longer names the net of U6.113 (USB1-DM)
- net USB1_D_P: no longer names the net of U6.112 (USB1-DP)
- net X32KIN: no longer names the net of U6.25 (X32KIN)
- net X32KOUT: no longer names the net of U6.24 (X32KOUT)
- new net: C18.1, C19.1, R36.1, U6.91 (AGND)
- no-connect marks 18 -> 0
Other:
- note removed: "T113-S3 的逐腳去耦（2026-10-10 補；mcu 頁手畫時漏了）"
- note removed: "★ 真正決定效果的是 layout：每一顆要貼著它負責的那支腳、via 直接下地平面。"
- note removed: "擺遠了就只是 BOM 上多幾顆料（概念 08）。"
- note removed: "每一條軌「幾支電源腳就幾顆 0.1uF」，核心與 DDR 另加 10uF 的本地 bulk。"

Commit message: wip
Parts:
- added C20, C21: 0.1uF, Capacitor_SMD:C_0603_1608Metric, symbol Device:C
- added C43, C44, C45, C46: 22pF, Capacitor_SMD:C_0603_1608Metric, symbol Device:C
- added C62, C63, C64, C65, C66, C68, C69, C72, C73, C74, C75, C76, C77, C78, C79, C80, C81, C82, C83, C84: 100nF, Capacitor_SMD:C_0603_1608Metric, symbol Device:C
- added C67, C70: 10uF, Capacitor_SMD:C_0805_2012Metric, symbol Device:C
- added C71: 2.2uF, Capacitor_SMD:C_0603_1608Metric, symbol Device:C
- added R37, R38: 33R, Resistor_SMD:R_0603_1608Metric, symbol Device:R
- added R39: 240R, Resistor_SMD:R_0603_1608Metric, symbol Device:R
- added Y2: 24MHz, Crystal:Crystal_SMD_2520-4Pin_2.5x2.0mm, symbol Device:Crystal_GND24
- added Y3: 32.768kHz, Crystal:Crystal_SMD_3215-2Pin_3.2x1.5mm, symbol Device:Crystal
- R20, R21, R22, R23, R24, R25, R26, R27, R28, R29, R30, R31, R32, R33, R34, R35, R36: footprint (none) -> Resistor_SMD:R_0603_1608Metric
- TP10, TP11, TP9: footprint Relay_THT:Relay_DPDT_Schrack-RT2-FormC_RM5mm -> TestPoint:TestPoint_Pad_D1.5mm
- U6: footprint (none) -> T113-DEV-V1:eLQFP-128_14x14mm_P0.4mm_EP5.72x5.72mm_ThermalVias
Connections:
- net +0V9: now also C62.1, C63.1, C64.1, C65.1, C66.1, C67.1
- net +1V5: now also C68.1, C69.1, C70.1
- net +1V8_AUDIO: now also C71.1, C72.1, C73.1
- net +1V8_SOC: now also C74.1, C75.1, C76.1, C77.1, C78.1
- net +3V3: now also C79.1, C80.1, C81.1, C82.1, C83.1, C84.1
- net GND: now also C18.1, C19.1, R36.1, U6.91 (AGND), C43.2, C44.2, C45.2, C46.2, C62.2, C63.2, C64.2, C65.2, C66.2, C67.2, C68.2, C69.2, C70.2, C71.2, C72.2, C73.2, C74.2, C75.2, C76.2, C77.2, C78.2, C79.2, C80.2, C81.2, C82.2, C83.2, C84.2, R39.1, Y2.2 (G), Y2.4 (G)
- net HP_FB: now reaches U6.100 (HPOUTFB)
- net at U6.98 (HPOUTR): now also R38.1
- net at U6.99 (HPOUTL): now also R37.1
- net USB1_D_P: now reaches U6.112 (USB1-DP)
- net USB1_D_N: now reaches U6.113 (USB1-DM)
- net USB0_D_N: now reaches U6.114 (USB0-DM)
- net USB0_D_P: now reaches U6.115 (USB0-DP)
- net DXOUT: now reaches U6.22 (DXOUT)
- net DXOUT: now also C44.1, Y2.3
- net DXIN: now reaches U6.23 (DXIN)
- net DXIN: now also C43.1, Y2.1
- net X32KOUT: now reaches U6.24 (X32KOUT)
- net X32KOUT: now also C46.1, Y3.2
- net X32KIN: now reaches U6.25 (X32KIN)
- net X32KIN: now also C45.1, Y3.1
- net SYS_RESET_N: now reaches U6.27 (RESET)
- net at U6.47 (DZQ): now also R39.2
- net DSI_CKN renamed DSI_CK_N
- net DSI_CKP renamed DSI_CK_P
- net DSI_D0N renamed DSI_D0_N
- net DSI_D0P renamed DSI_D0_P
- net DSI_D1N renamed DSI_D1_N
- net DSI_D1P renamed DSI_D1_P
- net DSI_D2N renamed DSI_D2_N
- net DSI_D2P renamed DSI_D2_P
- net DSI_D3N renamed DSI_D3_N
- net DSI_D3P renamed DSI_D3_P
- net HDR_GPIO7 renamed PANEL_RESET_N
- net HDR_GPIO8 renamed HDMI_INT_N
- net HDR_GPIO9 renamed HDMI_PD
- new net: C20.1, R37.2
- new net: C21.1, R38.2
- new net HP_L: C20.2
- new net HP_R: C21.2
- no-connect marks 0 -> 18
Other:
- note added: "T113-S3 的逐腳去耦（2026-10-10 補；mcu 頁手畫時漏了）"
- note added: "★ 真正決定效果的是 layout：每一顆要貼著它負責的那支腳、via 直接下地平面。"
- note added: "擺遠了就只是 BOM 上多幾顆料（概念 08）。"
- note added: "每一條軌「幾支電源腳就幾顆 0.1uF」，核心與 DDR 另加 10uF 的本地 bulk。"

Commit message: 還原,最終完整重跑
Parts:
- removed C20, C21: 0.1uF, Capacitor_SMD:C_0603_1608Metric, symbol Device:C
- removed C43, C44, C45, C46: 22pF, Capacitor_SMD:C_0603_1608Metric, symbol Device:C
- removed C62, C63, C64, C65, C66, C68, C69, C72, C73, C74, C75, C76, C77, C78, C79, C80, C81, C82, C83, C84: 100nF, Capacitor_SMD:C_0603_1608Metric, symbol Device:C
- removed C67, C70: 10uF, Capacitor_SMD:C_0805_2012Metric, symbol Device:C
- removed C71: 2.2uF, Capacitor_SMD:C_0603_1608Metric, symbol Device:C
- removed R37, R38: 33R, Resistor_SMD:R_0603_1608Metric, symbol Device:R
- removed R39: 240R, Resistor_SMD:R_0603_1608Metric, symbol Device:R
- removed Y2: 24MHz, Crystal:Crystal_SMD_2520-4Pin_2.5x2.0mm, symbol Device:Crystal_GND24
- removed Y3: 32.768kHz, Crystal:Crystal_SMD_3215-2Pin_3.2x1.5mm, symbol Device:Crystal
- R20, R21, R22, R23, R24, R25, R26, R27, R28, R29, R30, R31, R32, R33, R34, R35, R36: footprint Resistor_SMD:R_0603_1608Metric -> (none)
- TP10, TP11, TP9: footprint TestPoint:TestPoint_Pad_D1.5mm -> Relay_THT:Relay_DPDT_Schrack-RT2-FormC_RM5mm
- U6: footprint T113-DEV-V1:eLQFP-128_14x14mm_P0.4mm_EP5.72x5.72mm_ThermalVias -> (none)
Connections:
- net GND: no longer C18.1, C19.1, R36.1, U6.91 (AGND)
- net DSI_CK_N renamed DSI_CKN
- net DSI_CK_P renamed DSI_CKP
- net DSI_D0_N renamed DSI_D0N
- net DSI_D0_P renamed DSI_D0P
- net DSI_D1_N renamed DSI_D1N
- net DSI_D1_P renamed DSI_D1P
- net DSI_D2_N renamed DSI_D2N
- net DSI_D2_P renamed DSI_D2P
- net DSI_D3_N renamed DSI_D3N
- net DSI_D3_P renamed DSI_D3P
- net DXIN: no longer names the net of U6.23 (DXIN)
- net DXOUT: no longer names the net of U6.22 (DXOUT)
- net HDMI_INT_N renamed HDR_GPIO8
- net HDMI_PD renamed HDR_GPIO9
- net HP_FB: no longer names the net of U6.100 (HPOUTFB)
- net PANEL_RESET_N renamed HDR_GPIO7
- net SYS_RESET_N: no longer names the net of U6.27 (RESET)
- net USB0_D_N: no longer names the net of U6.114 (USB0-DM)
- net USB0_D_P: no longer names the net of U6.115 (USB0-DP)
- net USB1_D_N: no longer names the net of U6.113 (USB1-DM)
- net USB1_D_P: no longer names the net of U6.112 (USB1-DP)
- net X32KIN: no longer names the net of U6.25 (X32KIN)
- net X32KOUT: no longer names the net of U6.24 (X32KOUT)
- new net: C18.1, C19.1, R36.1, U6.91 (AGND)
- no-connect marks 18 -> 0
Other:
- note removed: "T113-S3 的逐腳去耦（2026-10-10 補；mcu 頁手畫時漏了）"
- note removed: "★ 真正決定效果的是 layout：每一顆要貼著它負責的那支腳、via 直接下地平面。"
- note removed: "擺遠了就只是 BOM 上多幾顆料（概念 08）。"
- note removed: "每一條軌「幾支電源腳就幾顆 0.1uF」，核心與 DDR 另加 10uF 的本地 bulk。"
